Commit message: franka test and remote control satellite panda connection tested

File: src/spaceman/src/assets/urdf/satellite_combine_panda/satellite_combine_panda.urdf (robot description, URDF)
Before this commit: robot satellite_combine_panda, 17 links, 16 joints
Joints:
- joint satellite_panda_connection_joint: origin xyz=0 0 1.0 rpy=0 0 0 -> xyz=-1 0 0 rpy=0 0 0
