Commit message: new Ros Node StarlinkManipulator and master_ee_control node

File: src/spaceman/src/assets/urdf/starlink_combine_qf_space_manipulator/starlink_combine_qf_space_manipulator.urdf (robot description, URDF)
Before this commit: robot starlink_combine_qf_space_manipulator, 15 links, 14 joints
Joints:
- joint qf_space_manipulator_joint2: origin xyz=-0.119999999999823 -0.0984119999999676 0.1079999999995944 rpy=0 0 0 -> xyz=-0.119999999999823 -0.0984119999999676 0.1079999999995944 rpy=0 -0.61 0
- joint qf_space_manipulator_joint3: origin xyz=0.4173123894383922 0.1314120000002838 0.586728531453288 rpy=0 0 0 -> xyz=0.4173123894383922 0.1314120000002838 0.586728531453288 rpy=0 -0.37 0
- joint qf_space_manipulator_joint4: origin xyz=-0.2799123894308418 -0.1266599999010702 0.4009614124181688 rpy=0 0 0 -> xyz=-0.2799123894308418 -0.1266599999010702 0.4009614124181688 rpy=0 -2.25 0
- joint qf_space_manipulator_joint5: origin xyz=0.0947999999922654 -0.106200000107286 0.0 rpy=0 0 0 -> xyz=0.0947999999922654 -0.106200000107286 0.0 rpy=-1.6 0 0
- joint starlink_qf_space_manipulator_connection_joint: origin xyz=-0.2 1.95 0 rpy=0 0 0 -> xyz=-0.87 1.05 0 rpy=0 0 1.574

Commit message: Add PID with gpu

File: src/spaceman/src/assets/urdf/starlink_combine_qf_space_manipulator/starlink_combine_qf_space_manipulator.urdf (robot description, URDF)
Before this commit: robot starlink_combine_qf_space_manipulator, 15 links, 14 joints
Links:
- removed link qf_space_manipulator_Link1
- removed link qf_space_manipulator_Link10
- removed link qf_space_manipulator_Link11
- removed link qf_space_manipulator_Link12
- removed link qf_space_manipulator_Link2
- removed link qf_space_manipulator_Link3
- removed link qf_space_manipulator_Link4
- removed link qf_space_manipulator_Link5
- removed link qf_space_manipulator_Link6
- removed link qf_space_manipulator_Link7
- removed link qf_space_manipulator_Link8
- removed link qf_space_manipulator_Link9
- added link qf_space_manipulator_2F-Body_Link, mass 0.08627345743213395; collision mesh filename=./meshes/2F-Body_Link.STL scale=0.6 0.6 0.6; visual mesh filename=./meshes/2F-Body_Link.STL scale=0.6 0.6 0.6
- added link qf_space_manipulator_Finger1_1_Link, mass 0.006898141207592574; collision mesh filename=./meshes/Finger1_1_Link.STL scale=0.6 0.6 0.6; visual mesh filename=./meshes/Finger1_1_Link.STL scale=0.6 0.6 0.6
- added link qf_space_manipulator_Finger1_2_Link, mass 0.006898141202937839; collision mesh filename=./meshes/Finger1_2_Link.STL scale=0.6 0.6 0.6; visual mesh filename=./meshes/Finger1_2_Link.STL scale=0.6 0.6 0.6
- added link qf_space_manipulator_Finger3_1_Link, mass 0.005448925989361684; collision mesh filename=./meshes/Finger3_1_Link.STL scale=0.6 0.6 0.6; visual mesh filename=./meshes/Finger3_1_Link.STL scale=0.6 0.6 0.6
- added link qf_space_manipulator_Finger3_2_Link, mass 0.005448926166982977; collision mesh filename=./meshes/Finger3_2_Link.STL scale=0.6 0.6 0.6; visual mesh filename=./meshes/Finger3_2_Link.STL scale=0.6 0.6 0.6
- added link qf_space_manipulator_Finger4_1_Link, mass 0.0015594313608905915; collision mesh filename=./meshes/Finger4_1_Link.STL scale=0.6 0.6 0.6; visual mesh filename=./meshes/Finger4_1_Link.STL scale=0.6 0.6 0.6
- added link qf_space_manipulator_Finger4_2_Link, mass 0.001559431360890557; collision mesh filename=./meshes/Finger4_2_Link.STL scale=0.6 0.6 0.6; visual mesh filename=./meshes/Finger4_2_Link.STL scale=0.6 0.6 0.6
- added link qf_space_manipulator_Mid_arm_Link_1, mass 4.394192754343932; collision mesh filename=./meshes/Mid_arm_Link_1.STL scale=0.6 0.6 0.6; visual mesh filename=./meshes/Mid_arm_Link_1.STL scale=0.6 0.6 0.6
- added link qf_space_manipulator_Shoulder_link_1, mass 1.1984038207793077; collision mesh filename=./meshes/Shoulder_link_1.STL scale=0.6 0.6 0.6; visual mesh filename=./meshes/Shoulder_link_1.STL scale=0.6 0.6 0.6
- added link qf_space_manipulator_Upper_arm_Link_1, mass 1.237014435999411; collision mesh filename=./meshes/Upper_arm_Link_1.STL scale=0.6 0.6 0.6; visual mesh filename=./meshes/Upper_arm_Link_1.STL scale=0.6 0.6 0.6
- added link qf_space_manipulator_Upper_wrist_Link_1, mass 0.30509485903504074; collision mesh filename=./meshes/Upper_wrist_Link_1.STL scale=0.6 0.6 0.6; visual mesh filename=./meshes/Upper_wrist_Link_1.STL scale=0.6 0.6 0.6
- added link qf_space_manipulator_Upper_wrist_Link_2, mass 0.3050948590124234; collision mesh filename=./meshes/Upper_wrist_Link_2.STL scale=0.6 0.6 0.6; visual mesh filename=./meshes/Upper_wrist_Link_2.STL scale=0.6 0.6 0.6
- link qf_space_manipulator_base_link: mass 2.080967403453504 -> 1.8705992689783575
Joints:
- removed joint qf_space_manipulator_joint1
- removed joint qf_space_manipulator_joint10
- removed joint qf_space_manipulator_joint11
- removed joint qf_space_manipulator_joint12
- removed joint qf_space_manipulator_joint2
- removed joint qf_space_manipulator_joint3
- removed joint qf_space_manipulator_joint4
- removed joint qf_space_manipulator_joint5
- removed joint qf_space_manipulator_joint6
- removed joint qf_space_manipulator_joint7
- removed joint qf_space_manipulator_joint8
- removed joint qf_space_manipulator_joint9
- added joint qf_space_manipulator_2F-Body_Link_pitch: type revolute, parent qf_space_manipulator_Upper_wrist_Link_2, child qf_space_manipulator_2F-Body_Link, origin xyz=-0.05819999999999988 -0.1008 0.0 rpy=0 1.5708 0, axis 0 -1 0, limit lower=0 upper=0 effort=0 velocity=0
- added joint qf_space_manipulator_Finger1_1_Link_roll: type revolute, parent qf_space_manipulator_2F-Body_Link, child qf_space_manipulator_Finger1_1_Link, origin xyz=0.00282 -0.0327978 -0.018360599999999998 rpy=0 0 0, axis -1 0 0, limit lower=0 upper=0 effort=0 velocity=0, mimic joint=qf_space_manipulator_Finger3_2_Link_roll multiplier=1 offset=0
- added joint qf_space_manipulator_Finger1_2_Link_roll: type revolute, parent qf_space_manipulator_2F-Body_Link, child qf_space_manipulator_Finger1_2_Link, origin xyz=0.00282 -0.0327978 0.018360599999999998 rpy=0 0 0, axis -1 0 0, limit lower=0 upper=0 effort=0 velocity=0, mimic joint=qf_space_manipulator_Finger3_2_Link_roll multiplier=-1 offset=0
- added joint qf_space_manipulator_Finger3_1_Link_roll: type revolute, parent qf_space_manipulator_2F-Body_Link, child qf_space_manipulator_Finger3_1_Link, origin xyz=0.006599999999999999 -0.0367068 -0.007619999999999999 rpy=0 0 0, axis 1 0 0, limit lower=0 upper=0 effort=0 velocity=0, mimic joint=qf_space_manipulator_Finger3_2_Link_roll multiplier=-1 offset=0
- added joint qf_space_manipulator_Finger3_2_Link_roll: type revolute, parent qf_space_manipulator_2F-Body_Link, child qf_space_manipulator_Finger3_2_Link, origin xyz=0.006599999999999999 -0.0367068 0.007619999999999999 rpy=0 0 0, axis 1 0 0, limit lower=0 upper=0 effort=0 velocity=0
- added joint qf_space_manipulator_Finger4_1_Link_roll: type revolute, parent qf_space_manipulator_Finger3_1_Link, child qf_space_manipulator_Finger4_1_Link, origin xyz=-0.0017399999999999998 -0.0520632 -0.0298236 rpy=0 0 0, axis -1 0 0, limit lower=0 upper=0 effort=0 velocity=0, mimic joint=qf_space_manipulator_Finger3_2_Link_roll multiplier=-1 offset=0
- added joint qf_space_manipulator_Finger4_2_Link_roll: type revolute, parent qf_space_manipulator_Finger3_2_Link, child qf_space_manipulator_Finger4_2_Link, origin xyz=-0.0018599999999999999 -0.051864 0.030168599999999997 rpy=0 0 0, axis 1 0 0, limit lower=0 upper=0 effort=0 velocity=0, mimic joint=qf_space_manipulator_Finger3_2_Link_roll multiplier=-1 offset=0
- added joint qf_space_manipulator_Mid_arm_Link_1_roll: type revolute, parent qf_space_manipulator_Upper_arm_Link_1, child qf_space_manipulator_Mid_arm_Link_1, origin xyz=-0.0054119999999258095 0.3426103217692296 0.63325995246783 rpy=0.22089323 0 0, axis -1 0 0, limit lower=0 upper=0 effort=0 velocity=0
- added joint qf_space_manipulator_Shoulder_link_1_yaw: type revolute, parent qf_space_manipulator_base_link, child qf_space_manipulator_Shoulder_link_1, origin xyz=0.0 0.0 0.138 rpy=0 0 0, axis 0 0 -1, limit lower=0 upper=0 effort=0 velocity=0
- added joint qf_space_manipulator_Upper_arm_Link_1_roll: type revolute, parent qf_space_manipulator_Shoulder_link_1, child qf_space_manipulator_Upper_arm_Link_1, origin xyz=0.0939119999999994 -0.1199999999999106 0.07800000000001318 rpy=0.49087385 0 0, axis 1 0 0, limit lower=0 upper=0 effort=0 velocity=0
- added joint qf_space_manipulator_Upper_wrist_Link_1_yaw: type revolute, parent qf_space_manipulator_Mid_arm_Link_1, child qf_space_manipulator_Upper_wrist_Link_1, origin xyz=0.0645000000001698 -0.4422422903588208 0.38137472592349375 rpy=0.859166812179351 0 0, axis 0 0 1, limit lower=0 upper=0 effort=0 velocity=0
- added joint qf_space_manipulator_Upper_wrist_Link_2_roll: type revolute, parent qf_space_manipulator_Upper_wrist_Link_1, child qf_space_manipulator_Upper_wrist_Link_2, origin xyz=-0.08760000000024659 0.0 0.058200000000027535 rpy=-1.5463902 0 0, axis 1 0 0, limit lower=0 upper=0 effort=0 velocity=0
- joint starlink_qf_space_manipulator_connection_joint: origin xyz=-0.87 1.05 0 rpy=0 0 1.574 -> xyz=-0.4 0.8 0 rpy=0 0 -1.574
